File: DC423-2018-Tracer/DC423-Tracer-V1.sch (KiCad schematic (older format))
At the start: 34 parts, among them J1 ISP Conn, U1 ATTINY841-SSU

Commit message: Final updates to schematic and added PDF of schematic
Other:
- note added: "2018-08"
- note added: "DC423 2018 Electronic Badge"
Changed lines of the file:
@@
 	1    0    0    -1
 $EndComp
+Text Notes 7400 7500 0    60   ~ 0
+DC423 2018 Electronic Badge
+Text Notes 8150 7650 0    60   ~ 0
+2018-08
 $EndSCHEMATC
